File: hardware/esp-4digit-display.sch (KiCad schematic (older format))
At the start: 21 parts, among them SW1 GP0, SW2 RST, U1 LM1117-3.3, U2 ESP-12, U3 74HC595

Commit message: Updated schematic with bit-to-digit mapping
Connections:
- no-connect marks 2 -> 1
Other:
- note added: "afbgedch"
Changed lines of the file:
@@
 	1    0    0    -1
-$EndComp
-$Comp
-L 74HC595 U3
-U 1 1 58BC92FD
-P 7150 5050
-F 0 "U3" H 7300 5650 50  0000 C CNN
-F 1 "74HC595" H 7150 4450 50  0000 C CNN
-F 2 "Housings_SOIC:SOIC-16_3.9x9.9mm_Pitch1.27mm" H 7150 5050 50  0001 C CNN
-F 3 "" H 7150 5050 50  0000 C CNN
-	1    7150 5050
-	0    -1   -1   0
 $EndComp
 NoConn ~ 7600 4350
-NoConn ~ 6850 5100
 $Comp
 L +3.3V #PWR03
@@
 	1    0    0    -1
 $EndComp
+$Comp
+L 74HC595 U3
+U 1 1 58BC92FD
+P 7150 5050
+F 0 "U3" H 7300 5650 50  0000 C CNN
+F 1 "74HC595" H 7150 4450 50  0000 C CNN
+F 2 "Housings_SOIC:SOIC-16_3.9x9.9mm_Pitch1.27mm" H 7150 5050 50  0001 C CNN
+F 3 "" H 7150 5050 50  0000 C CNN
+	1    7150 5050
+	0    -1   -1   0
+$EndComp
+Text Notes 6750 3850 0    60   ~ 12
+afbgedch
 $EndSCHEMATC
